Commit message: Add: Chassis and middle part ROS node

File: infantry_description/urdf/infantry.xacro (robot description, xacro)
@@ -24,5 +24,5 @@
   </collision>
 </link>
-<link name="SwervePart_2_1_1">
+<link name="SwervePart_4_1">
   <inertial>
     <origin rpy="0 0 0" xyz="0.00036972867304832513 0.0003204131523100451 0.010381504376103065"/>
@@ -33,5 +33,5 @@
     <origin rpy="0 0 0" xyz="-0.159993 0.16 -0.08165"/>
     <geometry>
-      <mesh filename="package://infantry_description/meshes/SwervePart_2_1_1.stl" scale="0.001 0.001 0.001"/>
+      <mesh filename="package://infantry_description/meshes/SwervePart_4_1.stl" scale="0.001 0.001 0.001"/>
     </geometry>
     <material name="silver"/>
@@ -40,5 +40,5 @@
     <origin rpy="0 0 0" xyz="-0.159993 0.16 -0.08165"/>
     <geometry>
-      <mesh filename="package://infantry_description/meshes/SwervePart_2_1_1.stl" scale="0.001 0.001 0.001"/>
+      <mesh filename="package://infantry_description/meshes/SwervePart_4_1.stl" scale="0.001 0.001 0.001"/>
     </geometry>
   </collision>
@@ -104,5 +104,5 @@
   </collision>
 </link>
-<link name="SwervePart_4_1">
+<link name="SwervePart_1_1">
   <inertial>
     <origin rpy="0 0 0" xyz="0.0003697278736722598 0.00032041395168808107 0.010381504376101802"/>
@@ -113,5 +113,5 @@
     <origin rpy="0 0 0" xyz="0.160007 -0.16 -0.08165"/>
     <geometry>
-      <mesh filename="package://infantry_description/meshes/SwervePart_4_1.stl" scale="0.001 0.001 0.001"/>
+      <mesh filename="package://infantry_description/meshes/SwervePart_1_1.stl" scale="0.001 0.001 0.001"/>
     </geometry>
     <material name="silver"/>
@@ -120,5 +120,5 @@
     <origin rpy="0 0 0" xyz="0.160007 -0.16 -0.08165"/>
     <geometry>
-      <mesh filename="package://infantry_description/meshes/SwervePart_4_1.stl" scale="0.001 0.001 0.001"/>
+      <mesh filename="package://infantry_description/meshes/SwervePart_1_1.stl" scale="0.001 0.001 0.001"/>
     </geometry>
   </collision>
@@ -144,5 +144,5 @@
   </collision>
 </link>
-<link name="SwervePart_1_1">
+<link name="SwervePart_2_1">
   <inertial>
     <origin rpy="0 0 0" xyz="-0.0003698802541624857 -0.0003200275145785747 0.010381504532545924"/>
@@ -153,5 +153,5 @@
     <origin rpy="0 0 0" xyz="-0.159993 -0.16 -0.08165"/>
     <geometry>
-      <mesh filename="package://infantry_description/meshes/SwervePart_1_1.stl" scale="0.001 0.001 0.001"/>
+      <mesh filename="package://infantry_description/meshes/SwervePart_2_1.stl" scale="0.001 0.001 0.001"/>
     </geometry>
     <material name="silver"/>
@@ -160,5 +160,5 @@
     <origin rpy="0 0 0" xyz="-0.159993 -0.16 -0.08165"/>
     <geometry>
-      <mesh filename="package://infantry_description/meshes/SwervePart_1_1.stl" scale="0.001 0.001 0.001"/>
+      <mesh filename="package://infantry_description/meshes/SwervePart_2_1.stl" scale="0.001 0.001 0.001"/>
     </geometry>
   </collision>
@@ -284,16 +284,45 @@
   </collision>
 </link>
+<!-- SWERVE: 27 29 31 33 -->
+<!-- Wheel:  28 30 32 34 -->
+<!--
+rostopic pub -r 1 /infantry/Rev27_position_controller/command std_msgs/Float64 "data: 0"
+rostopic pub -r 1 /infantry/Rev29_position_controller/command std_msgs/Float64 "data: 0"
+rostopic pub -r 1 /infantry/Rev31_position_controller/command std_msgs/Float64 "data: 0"
+rostopic pub -r 1 /infantry/Rev33_position_controller/command std_msgs/Float64 "data: 0"
+-->
+<!--
+rostopic pub -r 1 /infantry/Rev27_position_controller/command std_msgs/Float64 "data: 2.3562"
+rostopic pub -r 1 /infantry/Rev29_position_controller/command std_msgs/Float64 "data: 3.927"
+rostopic pub -r 1 /infantry/Rev31_position_controller/command std_msgs/Float64 "data: 5.49779"
+rostopic pub -r 1 /infantry/Rev33_position_controller/command std_msgs/Float64 "data: 0.7854"
+-->
+<!--
+rostopic pub -r 1 /infantry/Rev28_position_controller/command std_msgs/Float64 "data: 5"
+rostopic pub -r 1 /infantry/Rev30_position_controller/command std_msgs/Float64 "data: 5"
+rostopic pub -r 1 /infantry/Rev32_position_controller/command std_msgs/Float64 "data: 5"
+rostopic pub -r 1 /infantry/Rev34_position_controller/command std_msgs/Float64 "data: -5"
+-->
+<!--
+1/4 * pi = 0.7854
+2.3562
+3.927
+5.49779
+-->
+<!-- Swerve 4 RB -->
 <joint name="Rev27" type="continuous">
   <origin rpy="0 0 0" xyz="0.159993 -0.16 0.08165"/>
   <parent link="base_link"/>
-  <child link="SwervePart_2_1_1"/>
+  <child link="SwervePart_4_1"/>
   <axis xyz="-0.0 0.0 1.0"/>
 </joint>
+<!-- Wheel 4 RB -->
 <joint name="Rev28" type="continuous">
   <origin rpy="0 0 0" xyz="0.028 0.0 -0.04165"/>
-  <parent link="SwervePart_2_1_1"/>
+  <parent link="SwervePart_4_1"/>
   <child link="Wheel_4_1"/>
   <axis xyz="-1.0 -0.0 -0.0"/>
 </joint>
+<!-- Swerve 3 LB -->
 <joint name="Rev29" type="continuous">
   <origin rpy="0 0 0" xyz="-0.160007 -0.16 0.08165"/>
@@ -302,4 +331,5 @@
   <axis xyz="-0.0 0.0 1.0"/>
 </joint>
+<!-- Wheel 3 LB -->
 <joint name="Rev30" type="continuous">
   <origin rpy="0 0 0" xyz="0.028 0.0 -0.04165"/>
@@ -308,25 +338,29 @@
   <axis xyz="-1.0 -0.0 -0.0"/>
 </joint>
+<!-- Swerve 1 LF -->
 <joint name="Rev31" type="continuous">
   <origin rpy="0 0 0" xyz="-0.160007 0.16 0.08165"/>
   <parent link="base_link"/>
-  <child link="SwervePart_4_1"/>
+  <child link="SwervePart_1_1"/>
   <axis xyz="-0.0 0.0 1.0"/>
 </joint>
+<!-- Wheel 1 LF -->
 <joint name="Rev32" type="continuous">
   <origin rpy="0 0 0" xyz="0.028 0.0 -0.04165"/>
-  <parent link="SwervePart_4_1"/>
+  <parent link="SwervePart_1_1"/>
   <child link="Wheel_1_1"/>
   <axis xyz="-1.0 -0.0 -0.0"/>
 </joint>
+<!-- Swerve RF 2 -->
 <joint name="Rev33" type="continuous">
   <origin rpy="0 0 0" xyz="0.159993 0.16 0.08165"/>
   <parent link="base_link"/>
-  <child link="SwervePart_1_1"/>
+  <child link="SwervePart_2_1"/>
   <axis xyz="-0.0 0.0 1.0"/>
 </joint>
+<!-- Wheel RF 2 -->
 <joint name="Rev34" type="continuous">
   <origin rpy="0 0 0" xyz="0.028 0.0 -0.04165"/>
-  <parent link="SwervePart_1_1"/>
+  <parent link="SwervePart_2_1"/>
   <child link="Wheel_2_1"/>
   <axis xyz="-1.0 -0.0 -0.0"/>

Commit message: Add: infantry.xacro surface friction. Update: controller.yaml middlepart motor's pid

File: infantry_description/urdf/infantry.xacro (robot description, xacro)
@@ -4,4 +4,5 @@
 <xacro:include filename="$(find infantry_description)/urdf/infantry.trans" />
 <xacro:include filename="$(find infantry_description)/urdf/infantry.gazebo" />
+<!-- <link name="world"/> -->
 <link name="base_link">
   <inertial>
@@ -22,4 +23,12 @@
       <mesh filename="package://infantry_description/meshes/base_link.stl" scale="0.001 0.001 0.001"/>
     </geometry>
+    <surface>
+      <friction>
+        <ode>
+          <mu> 1.0 </mu>
+          <mu2> 1.0 </mu2>
+        </ode>
+      </friction>
+    </surface>
   </collision>
 </link>
@@ -42,4 +51,12 @@
       <mesh filename="package://infantry_description/meshes/SwervePart_4_1.stl" scale="0.001 0.001 0.001"/>
     </geometry>
+    <surface>
+      <friction>
+        <ode>
+          <mu> 1.0 </mu>
+          <mu2> 1.0 </mu2>
+        </ode>
+      </friction>
+    </surface>
   </collision>
 </link>
@@ -62,4 +79,12 @@
       <mesh filename="package://infantry_description/meshes/Wheel_4_1.stl" scale="0.001 0.001 0.001"/>
     </geometry>
+    <surface>
+      <friction>
+        <ode>
+          <mu> 1.0 </mu>
+          <mu2> 1.0 </mu2>
+        </ode>
+      </friction>
+    </surface>
   </collision>
 </link>
@@ -82,4 +107,12 @@
       <mesh filename="package://infantry_description/meshes/SwervePart_3_1.stl" scale="0.001 0.001 0.001"/>
     </geometry>
+    <surface>
+      <friction>
+        <ode>
+          <mu> 1.0 </mu>
+          <mu2> 1.0 </mu2>
+        </ode>
+      </friction>
+    </surface>
   </collision>
 </link>
@@ -102,4 +135,12 @@
       <mesh filename="package://infantry_description/meshes/Wheel_3_1.stl" scale="0.001 0.001 0.001"/>
     </geometry>
+    <surface>
+      <friction>
+        <ode>
+          <mu> 1.0 </mu>
+          <mu2> 1.0 </mu2>
+        </ode>
+      </friction>
+    </surface>
   </collision>
 </link>
@@ -122,4 +163,12 @@
       <mesh filename="package://infantry_description/meshes/SwervePart_1_1.stl" scale="0.001 0.001 0.001"/>
     </geometry>
+    <surface>
+      <friction>
+        <ode>
+          <mu> 1.0 </mu>
+          <mu2> 1.0 </mu2>
+        </ode>
+      </friction>
+    </surface>
   </collision>
 </link>
@@ -142,4 +191,12 @@
       <mesh filename="package://infantry_description/meshes/Wheel_1_1.stl" scale="0.001 0.001 0.001"/>
     </geometry>
+    <surface>
+      <friction>
+        <ode>
+          <mu> 1.0 </mu>
+          <mu2> 1.0 </mu2>
+        </ode>
+      </friction>
+    </surface>
   </collision>
 </link>
@@ -162,4 +219,12 @@
       <mesh filename="package://infantry_description/meshes/SwervePart_2_1.stl" scale="0.001 0.001 0.001"/>
     </geometry>
+    <surface>
+      <friction>
+        <ode>
+          <mu> 1.0 </mu>
+          <mu2> 1.0 </mu2>
+        </ode>
+      </friction>
+    </surface>
   </collision>
 </link>
@@ -182,4 +247,12 @@
       <mesh filename="package://infantry_description/meshes/Wheel_2_1.stl" scale="0.001 0.001 0.001"/>
     </geometry>
+    <surface>
+      <friction>
+        <ode>
+          <mu> 1.0 </mu>
+          <mu2> 1.0 </mu2>
+        </ode>
+      </friction>
+    </surface>
   </collision>
 </link>
@@ -202,4 +275,12 @@
       <mesh filename="package://infantry_description/meshes/GimbalMiddlePart_1.stl" scale="0.001 0.001 0.001"/>
     </geometry>
+    <surface>
+      <friction>
+        <ode>
+          <mu> 1.0 </mu>
+          <mu2> 1.0 </mu2>
+        </ode>
+      </friction>
+    </surface>
   </collision>
 </link>
@@ -222,4 +303,12 @@
       <mesh filename="package://infantry_description/meshes/Yaw_1.stl" scale="0.001 0.001 0.001"/>
     </geometry>
+    <surface>
+      <friction>
+        <ode>
+          <mu> 1.0 </mu>
+          <mu2> 1.0 </mu2>
+        </ode>
+      </friction>
+    </surface>
   </collision>
 </link>
@@ -242,4 +331,12 @@
       <mesh filename="package://infantry_description/meshes/Pitch_1.stl" scale="0.001 0.001 0.001"/>
     </geometry>
+    <surface>
+      <friction>
+        <ode>
+          <mu> 1.0 </mu>
+          <mu2> 1.0 </mu2>
+        </ode>
+      </friction>
+    </surface>
   </collision>
 </link>
@@ -262,4 +359,12 @@
       <mesh filename="package://infantry_description/meshes/RealsenseD455_1.stl" scale="0.001 0.001 0.001"/>
     </geometry>
+    <surface>
+      <friction>
+        <ode>
+          <mu> 1.0 </mu>
+          <mu2> 1.0 </mu2>
+        </ode>
+      </friction>
+    </surface>
   </collision>
 </link>
@@ -282,4 +387,12 @@
       <mesh filename="package://infantry_description/meshes/VT02_1.stl" scale="0.001 0.001 0.001"/>
     </geometry>
+    <surface>
+      <friction>
+        <ode>
+          <mu> 1.0 </mu>
+          <mu2> 1.0 </mu2>
+        </ode>
+      </friction>
+    </surface>
   </collision>
 </link>
