Commit message: Update: Change swerve id

File: infantry_description/urdf/infantry.xacro (robot description, xacro)
@@ -4,5 +4,4 @@
 <xacro:include filename="$(find infantry_description)/urdf/infantry.trans" />
 <xacro:include filename="$(find infantry_description)/urdf/infantry.gazebo" />
-<!-- <link name="world"/> -->
 <link name="base_link">
   <inertial>
@@ -33,5 +32,5 @@
   </collision>
 </link>
-<link name="SwervePart_4_1">
+<link name="SwervePart_3">
   <inertial>
     <origin rpy="0 0 0" xyz="0.00036972867304832513 0.0003204131523100451 0.010381504376103065"/>
@@ -42,5 +41,5 @@
     <origin rpy="0 0 0" xyz="-0.159993 0.16 -0.08165"/>
     <geometry>
-      <mesh filename="package://infantry_description/meshes/SwervePart_4_1.stl" scale="0.001 0.001 0.001"/>
+      <mesh filename="package://infantry_description/meshes/SwervePart_3.stl" scale="0.001 0.001 0.001"/>
     </geometry>
     <material name="silver"/>
@@ -49,17 +48,17 @@
     <origin rpy="0 0 0" xyz="-0.159993 0.16 -0.08165"/>
     <geometry>
-      <mesh filename="package://infantry_description/meshes/SwervePart_4_1.stl" scale="0.001 0.001 0.001"/>
-    </geometry>
-    <surface>
-      <friction>
-        <ode>
-          <mu> 1.0 </mu>
-          <mu2> 1.0 </mu2>
-        </ode>
-      </friction>
-    </surface>
-  </collision>
-</link>
-<link name="Wheel_4_1">
+      <mesh filename="package://infantry_description/meshes/SwervePart_3.stl" scale="0.001 0.001 0.001"/>
+    </geometry>
+    <surface>
+      <friction>
+        <ode>
+          <mu> 1.0 </mu>
+          <mu2> 1.0 </mu2>
+        </ode>
+      </friction>
+    </surface>
+  </collision>
+</link>
+<link name="Wheel_3">
   <inertial>
     <origin rpy="0 0 0" xyz="-0.027720338795959698 1.9284210200920526e-07 -3.3408852014027435e-07"/>
@@ -70,5 +69,5 @@
     <origin rpy="0 0 0" xyz="-0.187993 0.16 -0.04"/>
     <geometry>
-      <mesh filename="package://infantry_description/meshes/Wheel_4_1.stl" scale="0.001 0.001 0.001"/>
+      <mesh filename="package://infantry_description/meshes/Wheel_3.stl" scale="0.001 0.001 0.001"/>
     </geometry>
     <material name="silver"/>
@@ -77,17 +76,17 @@
     <origin rpy="0 0 0" xyz="-0.187993 0.16 -0.04"/>
     <geometry>
-      <mesh filename="package://infantry_description/meshes/Wheel_4_1.stl" scale="0.001 0.001 0.001"/>
-    </geometry>
-    <surface>
-      <friction>
-        <ode>
-          <mu> 1.0 </mu>
-          <mu2> 1.0 </mu2>
-        </ode>
-      </friction>
-    </surface>
-  </collision>
-</link>
-<link name="SwervePart_3_1">
+      <mesh filename="package://infantry_description/meshes/Wheel_3.stl" scale="0.001 0.001 0.001"/>
+    </geometry>
+    <surface>
+      <friction>
+        <ode>
+          <mu> 1.0 </mu>
+          <mu2> 1.0 </mu2>
+        </ode>
+      </friction>
+    </surface>
+  </collision>
+</link>
+<link name="SwervePart_2">
   <inertial>
     <origin rpy="0 0 0" xyz="-0.0003698810535431307 -0.00032002831395558373 0.010381504532544647"/>
@@ -98,5 +97,5 @@
     <origin rpy="0 0 0" xyz="0.160007 0.16 -0.08165"/>
     <geometry>
-      <mesh filename="package://infantry_description/meshes/SwervePart_3_1.stl" scale="0.001 0.001 0.001"/>
+      <mesh filename="package://infantry_description/meshes/SwervePart_2.stl" scale="0.001 0.001 0.001"/>
     </geometry>
     <material name="silver"/>
@@ -105,17 +104,17 @@
     <origin rpy="0 0 0" xyz="0.160007 0.16 -0.08165"/>
     <geometry>
-      <mesh filename="package://infantry_description/meshes/SwervePart_3_1.stl" scale="0.001 0.001 0.001"/>
-    </geometry>
-    <surface>
-      <friction>
-        <ode>
-          <mu> 1.0 </mu>
-          <mu2> 1.0 </mu2>
-        </ode>
-      </friction>
-    </surface>
-  </collision>
-</link>
-<link name="Wheel_3_1">
+      <mesh filename="package://infantry_description/meshes/SwervePart_2.stl" scale="0.001 0.001 0.001"/>
+    </geometry>
+    <surface>
+      <friction>
+        <ode>
+          <mu> 1.0 </mu>
+          <mu2> 1.0 </mu2>
+        </ode>
+      </friction>
+    </surface>
+  </collision>
+</link>
+<link name="Wheel_2">
   <inertial>
     <origin rpy="0 0 0" xyz="-0.02827981358383913 1.9284210189818296e-07 -3.340885198696575e-07"/>
@@ -126,5 +125,5 @@
     <origin rpy="0 0 0" xyz="0.132007 0.16 -0.04"/>
     <geometry>
-      <mesh filename="package://infantry_description/meshes/Wheel_3_1.stl" scale="0.001 0.001 0.001"/>
+      <mesh filename="package://infantry_description/meshes/Wheel_2.stl" scale="0.001 0.001 0.001"/>
     </geometry>
     <material name="silver"/>
@@ -133,17 +132,17 @@
     <origin rpy="0 0 0" xyz="0.132007 0.16 -0.04"/>
     <geometry>
-      <mesh filename="package://infantry_description/meshes/Wheel_3_1.stl" scale="0.001 0.001 0.001"/>
-    </geometry>
-    <surface>
-      <friction>
-        <ode>
-          <mu> 1.0 </mu>
-          <mu2> 1.0 </mu2>
-        </ode>
-      </friction>
-    </surface>
-  </collision>
-</link>
-<link name="SwervePart_1_1">
+      <mesh filename="package://infantry_description/meshes/Wheel_2.stl" scale="0.001 0.001 0.001"/>
+    </geometry>
+    <surface>
+      <friction>
+        <ode>
+          <mu> 1.0 </mu>
+          <mu2> 1.0 </mu2>
+        </ode>
+      </friction>
+    </surface>
+  </collision>
+</link>
+<link name="SwervePart_0">
   <inertial>
     <origin rpy="0 0 0" xyz="0.0003697278736722598 0.00032041395168808107 0.010381504376101802"/>
@@ -154,5 +153,5 @@
     <origin rpy="0 0 0" xyz="0.160007 -0.16 -0.08165"/>
     <geometry>
-      <mesh filename="package://infantry_description/meshes/SwervePart_1_1.stl" scale="0.001 0.001 0.001"/>
+      <mesh filename="package://infantry_description/meshes/SwervePart_0.stl" scale="0.001 0.001 0.001"/>
     </geometry>
     <material name="silver"/>
@@ -161,17 +160,17 @@
     <origin rpy="0 0 0" xyz="0.160007 -0.16 -0.08165"/>
     <geometry>
-      <mesh filename="package://infantry_description/meshes/SwervePart_1_1.stl" scale="0.001 0.001 0.001"/>
-    </geometry>
-    <surface>
-      <friction>
-        <ode>
-          <mu> 1.0 </mu>
-          <mu2> 1.0 </mu2>
-        </ode>
-      </friction>
-    </surface>
-  </collision>
-</link>
-<link name="Wheel_1_1">
+      <mesh filename="package://infantry_description/meshes/SwervePart_0.stl" scale="0.001 0.001 0.001"/>
+    </geometry>
+    <surface>
+      <friction>
+        <ode>
+          <mu> 1.0 </mu>
+          <mu2> 1.0 </mu2>
+        </ode>
+      </friction>
+    </surface>
+  </collision>
+</link>
+<link name="Wheel_0">
   <inertial>
     <origin rpy="0 0 0" xyz="-0.028279813583838742 1.9284210203696084e-07 -3.340885198419019e-07"/>
@@ -182,5 +181,5 @@
     <origin rpy="0 0 0" xyz="0.132007 -0.16 -0.04"/>
     <geometry>
-      <mesh filename="package://infantry_description/meshes/Wheel_1_1.stl" scale="0.001 0.001 0.001"/>
+      <mesh filename="package://infantry_description/meshes/Wheel_0.stl" scale="0.001 0.001 0.001"/>
     </geometry>
     <material name="silver"/>
@@ -189,17 +188,17 @@
     <origin rpy="0 0 0" xyz="0.132007 -0.16 -0.04"/>
     <geometry>
-      <mesh filename="package://infantry_description/meshes/Wheel_1_1.stl" scale="0.001 0.001 0.001"/>
-    </geometry>
-    <surface>
-      <friction>
-        <ode>
-          <mu> 1.0 </mu>
-          <mu2> 1.0 </mu2>
-        </ode>
-      </friction>
-    </surface>
-  </collision>
-</link>
-<link name="SwervePart_2_1">
+      <mesh filename="package://infantry_description/meshes/Wheel_0.stl" scale="0.001 0.001 0.001"/>
+    </geometry>
+    <surface>
+      <friction>
+        <ode>
+          <mu> 1.0 </mu>
+          <mu2> 1.0 </mu2>
+        </ode>
+      </friction>
+    </surface>
+  </collision>
+</link>
+<link name="SwervePart_1">
   <inertial>
     <origin rpy="0 0 0" xyz="-0.0003698802541624857 -0.0003200275145785747 0.010381504532545924"/>
@@ -210,5 +209,5 @@
     <origin rpy="0 0 0" xyz="-0.159993 -0.16 -0.08165"/>
     <geometry>
-      <mesh filename="package://infantry_description/meshes/SwervePart_2_1.stl" scale="0.001 0.001 0.001"/>
+      <mesh filename="package://infantry_description/meshes/SwervePart_1.stl" scale="0.001 0.001 0.001"/>
     </geometry>
     <material name="silver"/>
@@ -217,17 +216,17 @@
     <origin rpy="0 0 0" xyz="-0.159993 -0.16 -0.08165"/>
     <geometry>
-      <mesh filename="package://infantry_description/meshes/SwervePart_2_1.stl" scale="0.001 0.001 0.001"/>
-    </geometry>
-    <surface>
-      <friction>
-        <ode>
-          <mu> 1.0 </mu>
-          <mu2> 1.0 </mu2>
-        </ode>
-      </friction>
-    </surface>
-  </collision>
-</link>
-<link name="Wheel_2_1">
+      <mesh filename="package://infantry_description/meshes/SwervePart_1.stl" scale="0.001 0.001 0.001"/>
+    </geometry>
+    <surface>
+      <friction>
+        <ode>
+          <mu> 1.0 </mu>
+          <mu2> 1.0 </mu2>
+        </ode>
+      </friction>
+    </surface>
+  </collision>
+</link>
+<link name="Wheel_1">
   <inertial>
     <origin rpy="0 0 0" xyz="-0.02772033879595956 1.9284210125980472e-07 -3.340885201055799e-07"/>
@@ -238,5 +237,5 @@
     <origin rpy="0 0 0" xyz="-0.187993 -0.16 -0.04"/>
     <geometry>
-      <mesh filename="package://infantry_description/meshes/Wheel_2_1.stl" scale="0.001 0.001 0.001"/>
+      <mesh filename="package://infantry_description/meshes/Wheel_1.stl" scale="0.001 0.001 0.001"/>
     </geometry>
     <material name="silver"/>
@@ -245,5 +244,5 @@
     <origin rpy="0 0 0" xyz="-0.187993 -0.16 -0.04"/>
     <geometry>
-      <mesh filename="package://infantry_description/meshes/Wheel_2_1.stl" scale="0.001 0.001 0.001"/>
+      <mesh filename="package://infantry_description/meshes/Wheel_1.stl" scale="0.001 0.001 0.001"/>
     </geometry>
     <surface>
@@ -399,82 +398,58 @@
 <!-- SWERVE: 27 29 31 33 -->
 <!-- Wheel:  28 30 32 34 -->
-<!--
-rostopic pub -r 1 /infantry/Rev27_position_controller/command std_msgs/Float64 "data: 0"
-rostopic pub -r 1 /infantry/Rev29_position_controller/command std_msgs/Float64 "data: 0"
-rostopic pub -r 1 /infantry/Rev31_position_controller/command std_msgs/Float64 "data: 0"
-rostopic pub -r 1 /infantry/Rev33_position_controller/command std_msgs/Float64 "data: 0"
--->
-<!--
-rostopic pub -r 1 /infantry/Rev27_position_controller/command std_msgs/Float64 "data: 2.3562"
-rostopic pub -r 1 /infantry/Rev29_position_controller/command std_msgs/Float64 "data: 3.927"
-rostopic pub -r 1 /infantry/Rev31_position_controller/command std_msgs/Float64 "data: 5.49779"
-rostopic pub -r 1 /infantry/Rev33_position_controller/command std_msgs/Float64 "data: 0.7854"
--->
-<!--
-rostopic pub -r 1 /infantry/Rev28_position_controller/command std_msgs/Float64 "data: 5"
-rostopic pub -r 1 /infantry/Rev30_position_controller/command std_msgs/Float64 "data: 5"
-rostopic pub -r 1 /infantry/Rev32_position_controller/command std_msgs/Float64 "data: 5"
-rostopic pub -r 1 /infantry/Rev34_position_controller/command std_msgs/Float64 "data: -5"
--->
-<!--
-1/4 * pi = 0.7854
-2.3562
-3.927
-5.49779
--->
-<!-- Swerve 4 RB -->
+<!-- Swerve 3 RB -->
 <joint name="Rev27" type="continuous">
   <origin rpy="0 0 0" xyz="0.159993 -0.16 0.08165"/>
   <parent link="base_link"/>
-  <child link="SwervePart_4_1"/>
+  <child link="SwervePart_3"/>
   <axis xyz="-0.0 0.0 1.0"/>
 </joint>
-<!-- Wheel 4 RB -->
+<!-- Wheel 3 RB -->
 <joint name="Rev28" type="continuous">
   <origin rpy="0 0 0" xyz="0.028 0.0 -0.04165"/>
-  <parent link="SwervePart_4_1"/>
-  <child link="Wheel_4_1"/>
+  <parent link="SwervePart_3"/>
+  <child link="Wheel_3"/>
   <axis xyz="-1.0 -0.0 -0.0"/>
 </joint>
-<!-- Swerve 3 LB -->
+<!-- Swerve 2 LB -->
 <joint name="Rev29" type="continuous">
   <origin rpy="0 0 0" xyz="-0.160007 -0.16 0.08165"/>
   <parent link="base_link"/>
-  <child link="SwervePart_3_1"/>
+  <child link="SwervePart_2"/>
   <axis xyz="-0.0 0.0 1.0"/>
 </joint>
-<!-- Wheel 3 LB -->
+<!-- Wheel 2 LB -->
 <joint name="Rev30" type="continuous">
   <origin rpy="0 0 0" xyz="0.028 0.0 -0.04165"/>
-  <parent link="SwervePart_3_1"/>
-  <child link="Wheel_3_1"/>
+  <parent link="SwervePart_2"/>
+  <child link="Wheel_2"/>
   <axis xyz="-1.0 -0.0 -0.0"/>
 </joint>
-<!-- Swerve 1 LF -->
+<!-- Swerve 0 LF -->
 <joint name="Rev31" type="continuous">
   <origin rpy="0 0 0" xyz="-0.160007 0.16 0.08165"/>
   <parent link="base_link"/>
-  <child link="SwervePart_1_1"/>
+  <child link="SwervePart_0"/>
   <axis xyz="-0.0 0.0 1.0"/>
 </joint>
-<!-- Wheel 1 LF -->
+<!-- Wheel 0 LF -->
 <joint name="Rev32" type="continuous">
   <origin rpy="0 0 0" xyz="0.028 0.0 -0.04165"/>
-  <parent link="SwervePart_1_1"/>
-  <child link="Wheel_1_1"/>
+  <parent link="SwervePart_0"/>
+  <child link="Wheel_0"/>
   <axis xyz="-1.0 -0.0 -0.0"/>
 </joint>
-<!-- Swerve RF 2 -->
+<!-- Swerve RF 1 -->
 <joint name="Rev33" type="continuous">
   <origin rpy="0 0 0" xyz="0.159993 0.16 0.08165"/>
   <parent link="base_link"/>
-  <child link="SwervePart_2_1"/>
+  <child link="SwervePart_1"/>
   <axis xyz="-0.0 0.0 1.0"/>
 </joint>
-<!-- Wheel RF 2 -->
+<!-- Wheel RF 1 -->
 <joint name="Rev34" type="continuous">
   <origin rpy="0 0 0" xyz="0.028 0.0 -0.04165"/>
-  <parent link="SwervePart_2_1"/>
-  <child link="Wheel_2_1"/>
+  <parent link="SwervePart_1"/>
+  <child link="Wheel_1"/>
   <axis xyz="-1.0 -0.0 -0.0"/>
 </joint>

Commit message: Fix: Motion control; Add: SLAM; Update: README.md

File: infantry_description/urdf/infantry.xacro (robot description, xacro)
@@ -4,4 +4,9 @@
 <xacro:include filename="$(find infantry_description)/urdf/infantry.trans" />
 <xacro:include filename="$(find infantry_description)/urdf/infantry.gazebo" />
+<!-- 为什么所有的模型都歪了90度？吐了！ -->
+<xacro:property name="model_tf_offset" value="-1.5707963267948965579989817342720925807952880859375" />
+<!-- ${model_tf_offset} -->
+<!-- <origin rpy="0 0 0 -->
+<!-- <origin rpy="0 0 ${model_tf_offset} -->
 <link name="base_link">
   <inertial>

File: infantry_description/urdf/infantry_sensor.xacro (robot description, xacro)
@@ -4,12 +4,14 @@
 <xacro:include filename="$(find infantry_description)/urdf/lidar.xacro"/>
     <xacro:property name="lidar_offset_x" value="0" />
-    <xacro:property name="lidar_offset_y" value="0.2" />
-    <xacro:property name="lidar_offset_z" value="0.25" />
-    <xacro:property name="lidar_offset_yaw" value="1.5707963267948966" /> <!-- PI / 2 -->
+    <xacro:property name="lidar_offset_y" value="0" />
+    <xacro:property name="lidar_offset_z" value="0.1" />
+    <!-- <xacro:property name="lidar_offset_yaw" value="1.5707963267948966" /> -->
     <!-- Lidar -->
     <joint name="lidar_joint" type="fixed">
         <origin xyz="${lidar_offset_x} ${lidar_offset_y} ${lidar_offset_z}"
-                rpy="0 0 ${lidar_offset_yaw}" />
-        <parent link="base_link"/>
+                rpy="0 0 0" />
+        <!-- <origin xyz="${lidar_offset_x} ${lidar_offset_y} ${lidar_offset_z}"
+                rpy="0 0 ${lidar_offset_yaw}" /> -->
+        <parent link="GimbalMiddlePart_1"/>
         <child link="laser_link"/>
     </joint>

File: infantry_description/urdf/lidar.xacro (robot description, xacro)
@@ -43,5 +43,5 @@
                     </scan>
                     <range>
-                      <min>0.10</min>
+                      <min>0.4</min>
                       <max>6.0</max>
                       <resolution>0.01</resolution>
