Commit message: Add: IMU; Update: Robust navigation

File: infantry_description/urdf/infantry_sensor.xacro (robot description, xacro)
@@ -1,6 +1,7 @@
 <?xml version="1.0"?>
-<robot name="arm" xmlns:xacro="http://www.ros.org/wiki/xacro">
+<robot name="infantry" xmlns:xacro="http://www.ros.org/wiki/xacro">
 <xacro:include filename="$(find infantry_description)/urdf/infantry.xacro" />
 <xacro:include filename="$(find infantry_description)/urdf/lidar.xacro"/>
+<xacro:include filename="$(find infantry_description)/urdf/imu.xacro"/>
     <xacro:property name="lidar_offset_x" value="0" />
     <xacro:property name="lidar_offset_y" value="0" />
@@ -16,4 +17,19 @@
         <child link="laser_link"/>
     </joint>
-    <xacro:lidar prefix="laser"/>
+    <!-- <xacro:lidar prefix="laser"/> -->
+    <xacro:property name="imu_offset_x" value="0" />
+    <xacro:property name="imu_offset_y" value="0" />
+    <!-- <xacro:property name="imu_offset_z" value="0.14" /> -->
+    <xacro:property name="imu_offset_z" value="0" />
+    <!-- <xacro:property name="imu_offset_yaw" value="1.5707963267948966" /> -->
+    <!-- IMU -->
+    <joint name="imu_joint" type="fixed">
+        <origin xyz="${imu_offset_x} ${imu_offset_y} ${imu_offset_z}"
+                rpy="0 0 0" />
+        <!-- <origin xyz="${imu_offset_x} ${imu_offset_y} ${imu_offset_z}"
+                rpy="0 0 ${imu_offset_yaw}" /> -->
+        <parent link="GimbalMiddlePart_1"/>
+        <child link="imu_link"/>
+    </joint>
+    <!-- <xacro:imu prefix="imu"/> -->
 </robot>

File: infantry_description/urdf/lidar.xacro (robot description, xacro)
@@ -1,62 +1,59 @@
 <?xml version="1.0"?>
-<robot xmlns:xacro="http://www.ros.org/wiki/xacro" name="laser">
-    <xacro:macro name="lidar" params="prefix:=laser">
-        <!-- Create laser reference frame -->
-        <link name="${prefix}_link">
-            <inertial>
-                <mass value="0.1" />
-                <origin xyz="0 0 0" />
-                <inertia ixx="0.01" ixy="0.0" ixz="0.0"
-                         iyy="0.01" iyz="0.0"
-                         izz="0.01" />
-            </inertial>
-            <visual>
-                <origin xyz=" 0 0 0 " rpy="0 0 0" />
-                <geometry>
-                    <cylinder length="0.05" radius="0.05"/>
-                </geometry>
-                <material name="black"/>
-            </visual>
-            <collision>
-                <origin xyz="0.0 0.0 0.0" rpy="0 0 0" />
-                <geometry>
-                    <cylinder length="0.06" radius="0.05"/>
-                </geometry>
-            </collision>
-        </link>
-        <gazebo reference="${prefix}_link">
-            <material>Gazebo/Black</material>
-        </gazebo>
-        <gazebo reference="${prefix}_link">
-            <sensor type="ray" name="lidar">
-                <pose>0 0 0 0 0 0</pose>
-                <visualize>false</visualize>
-                <update_rate>5.5</update_rate>
-                <ray>
-                    <scan>
-                      <horizontal>
-                        <samples>360</samples>
-                        <resolution>1</resolution>
-                        <min_angle>-3</min_angle>
-                        <max_angle>3</max_angle>
-                      </horizontal>
-                    </scan>
-                    <range>
-                      <min>0.4</min>
-                      <max>6.0</max>
-                      <resolution>0.01</resolution>
-                    </range>
-                    <noise>
-                      <type>gaussian</type>
-                      <mean>0.0</mean>
-                      <stddev>0.01</stddev>
-                    </noise>
-                </ray>
-                <plugin name="gazebo_lidar" filename="libgazebo_ros_laser.so">
-                    <topicName>/scan</topicName>
-                    <frameName>laser_link</frameName>
-                </plugin>
-            </sensor>
-        </gazebo>
-    </xacro:macro>
+<robot name="lidar" xmlns:xacro="http://www.ros.org/wiki/xacro">
+    <!-- Create laser reference frame -->
+    <link name="laser_link">
+        <inertial>
+            <mass value="0.1" />
+            <origin xyz="0 0 0" />
+            <inertia ixx="0.01" ixy="0.0" ixz="0.0"
+                        iyy="0.01" iyz="0.0"
+                        izz="0.01" />
+        </inertial>
+        <visual>
+            <origin xyz=" 0 0 0 " rpy="0 0 0" />
+            <geometry>
+                <cylinder length="0.04" radius="0.04"/>
+            </geometry>
+            <material name="black"/>
+        </visual>
+        <collision>
+            <origin xyz="0.0 0.0 0.0" rpy="0 0 0" />
+            <geometry>
+                <cylinder length="0.04" radius="0.04"/>
+            </geometry>
+        </collision>
+    </link>
+    <!-- 使用rplidarA2参数 -->
+    <gazebo reference="laser_link">
+        <material>Gazebo/Black</material>
+        <sensor name="lidar" type="ray">
+            <pose>0 0 0 0 0 0</pose>
+            <visualize>false</visualize>
+            <update_rate>10</update_rate>
+            <ray>
+                <scan>
+                    <horizontal>
+                    <samples>400</samples>
+                    <resolution>0.9</resolution>
+                    <min_angle>-3.14159265359</min_angle>
+                    <max_angle>3.14159265359</max_angle>
+                    </horizontal>
+                </scan>
+                <range>
+                    <min>0.3</min>
+                    <max>12</max> <!-- 测距距离仅保留分辨率为1%的部分 -->
+                    <resolution>0.01</resolution>
+                </range>
+                <noise>
+                    <type>gaussian</type>
+                    <mean>0.0</mean>
+                    <stddev>0.01</stddev>
+                </noise>
+            </ray>
+            <plugin name="gazebo_lidar" filename="libgazebo_ros_laser.so">
+                <topicName>/scan</topicName>
+                <frameName>laser_link</frameName>
+            </plugin>
+        </sensor>
+    </gazebo>
 </robot>

Commit message: Add: Serial port communication

File: infantry_description/urdf/infantry_sensor.xacro (robot description, xacro)
@@ -2,6 +2,6 @@
 <robot name="infantry" xmlns:xacro="http://www.ros.org/wiki/xacro">
 <xacro:include filename="$(find infantry_description)/urdf/infantry.xacro" />
-<xacro:include filename="$(find infantry_description)/urdf/lidar.xacro"/>
-<xacro:include filename="$(find infantry_description)/urdf/imu.xacro"/>
+<!-- <xacro:include filename="$(find infantry_description)/urdf/lidar.xacro"/> -->
+<!-- <xacro:include filename="$(find infantry_description)/urdf/imu.xacro"/> -->
     <xacro:property name="lidar_offset_x" value="0" />
     <xacro:property name="lidar_offset_y" value="0" />
@@ -9,12 +9,12 @@
     <!-- <xacro:property name="lidar_offset_yaw" value="1.5707963267948966" /> -->
     <!-- Lidar -->
-    <joint name="lidar_joint" type="fixed">
+    <!-- <joint name="lidar_joint" type="fixed">
         <origin xyz="${lidar_offset_x} ${lidar_offset_y} ${lidar_offset_z}"
-                rpy="0 0 0" />
+                rpy="0 0 0" /> -->
         <!-- <origin xyz="${lidar_offset_x} ${lidar_offset_y} ${lidar_offset_z}"
                 rpy="0 0 ${lidar_offset_yaw}" /> -->
-        <parent link="GimbalMiddlePart_1"/>
+        <!-- <parent link="GimbalMiddlePart_1"/>
         <child link="laser_link"/>
-    </joint>
+    </joint> -->
     <!-- <xacro:lidar prefix="laser"/> -->
     <xacro:property name="imu_offset_x" value="0" />
@@ -24,12 +24,12 @@
     <!-- <xacro:property name="imu_offset_yaw" value="1.5707963267948966" /> -->
     <!-- IMU -->
-    <joint name="imu_joint" type="fixed">
+    <!-- <joint name="imu_joint" type="fixed">
         <origin xyz="${imu_offset_x} ${imu_offset_y} ${imu_offset_z}"
-                rpy="0 0 0" />
+                rpy="0 0 0" /> -->
         <!-- <origin xyz="${imu_offset_x} ${imu_offset_y} ${imu_offset_z}"
                 rpy="0 0 ${imu_offset_yaw}" /> -->
-        <parent link="GimbalMiddlePart_1"/>
+        <!-- <parent link="GimbalMiddlePart_1"/>
         <child link="imu_link"/>
-    </joint>
+    </joint> -->
     <!-- <xacro:imu prefix="imu"/> -->
 </robot>
